File: ECAD Files/EAGLE Files/Thanics Halo/Flight Controller Auxiliary Board/Flight Controller Auxiliary Board.brd (EAGLE design)
At the start: 58.5 x 28.4 mm, 48 parts, among them J3 MAGJACK, U3 WGM110A

Commit message: Reorganized ECAD Files
Parts:
- moved C24 7.95 mm to (54.3, 47.4), flipped to the top, turned to 90 degrees
- moved R4 1.38 mm to (50.3, 46.9), turned to 270 degrees
- moved C20 0.77 mm to (48.4, 39.4), turned to 90 degrees
- moved R3 0.76 mm to (49.1, 45.5), turned to 315 degrees
- moved R6 0.57 mm to (50.9, 46.3), turned to 315 degrees
- moved C19 0.31 mm to (52.5, 40.9)
Routing:
- net USB_D2_P: track 27.4 -> 35.0 mm
- net USB_D2_N: track 27.3 -> 34.9 mm
- net GND: track 27.4 -> 31.1 mm, vias 18 -> 25
- net RX_N: track 30.0 -> 28.0 mm
- net 3.3V_A: track 55.2 -> 57.1 mm
- net RX_P: track 28.5 -> 26.6 mm
- net TX_P: track 26.5 -> 25.3 mm
- net USB_D3_P: track 22.7 -> 21.7 mm
- net +5V: track 23.7 -> 24.5 mm, vias 1 -> 2
- net USB_D_N: track 7.05 -> 6.24 mm
- net USB_D_P: track 7.49 -> 6.77 mm
- added copper zone on layer 2, net +3V3
- added copper zone on layer 15, net GND
- added copper zone on layer 16, net N$5
